File: one-shift-register.kicad_pcb (KiCad board)
At the start: 2 copper layers, 68.6 x 53.3 mm, 25 parts, among them P1 Power, P2 Analog, P3 Digital, P4 Digital, P5 CONN_1, P6 CONN_1, P7 CONN_1, P8 CONN_1, U1 74HC595

Commit message: added text to PCB; turned on all arduino demos
Other:
- board text added: "Marginallyclever.com 2017-02-14 ELEC-0122 shift register LED demo"
Changed lines of the file:
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@@
     (area 110.922999 72.949999 179.653001 126.440001)
     (thickness 1.6)
-    (drawings 27)
+    (drawings 28)
     (tracks 50)
     (zones 0)
@@
     (nets 52)
   )
-  (page A4)
+  (page USLetter)
   (title_block
-    (date "lun. 30 mars 2015")
+    (title "ELEC-0122 shift register LED demo PCB")
+    (date 2017-02-14)
+    (rev 2)
+    (company Marginallyclever.com)
+    (comment 1 "Dan Royer (dan@marginallyclever.com)")
   )
   (layers
-    (0 F.Cu signal)
-    (31 B.Cu signal)
+    (0 F.Cu signal hide)
+    (31 B.Cu signal hide)
     (32 B.Adhes user)
     (33 F.Adhes user)
@@
     )
   )
+  (gr_text "Marginallyclever.com 2017-02-14\nELEC-0122 shift register LED demo\n" (at 120.65 99.441 90) (layer F.Mask)
+    (effects (font (size 1.5 1.5) (thickness 0.3)))
+  )
   (gr_text 1 (at 138.938 121.285 90) (layer F.SilkS)
     (effects (font (size 1 1) (thickness 0.15)))
@@
   (gr_line (start 120.523 82.55) (end 120.523 93.98) (angle 90) (layer Dwgs.User) (width 0.15))
   (gr_line (start 104.648 82.55) (end 120.523 82.55) (angle 90) (layer Dwgs.User) (width 0.15))
-  (segment (start 159.258 75.565) (end 156.21 78.613) (width 0.25) (layer F.Cu) (net 16) (status 400000))
-  (segment (start 153.035 78.613) (end 146.558 85.09) (width 0.25) (layer F.Cu) (net 16) (status 800000))
+  (segment (start 159.258 75.565) (end 156.21 78.613) (width 0.25) (layer F.Cu) (net 16))
+  (segment (start 153.035 78.613) (end 146.558 85.09) (width 0.25) (layer F.Cu) (net 16))
   (segment (start 156.21 78.613) (end 153.035 78.613) (width 0.25) (layer F.Cu) (net 16))
-  (segment (start 161.798 75.565) (end 161.798 77.47) (width 0.25) (layer F.Cu) (net 17) (status 400000))
-  (segment (start 161.798 77.47) (end 154.178 85.09) (width 0.25) (layer F.Cu) (net 17) (status 800000))
-  (segment (start 164.338 75.565) (end 164.338 77.47) (width 0.25) (layer F.Cu) (net 18) (status 400000))
-  (segment (start 164.338 77.47) (end 156.718 85.09) (width 0.25) (layer F.Cu) (net 18) (status 800000))
-  (segment (start 166.878 75.565) (end 166.878 81.661) (width 0.25) (layer F.Cu) (net 19) (status 400000))
-  (segment (start 153.797 87.249) (end 151.638 85.09) (width 0.25) (layer F.Cu) (net 19) (status 800000))
+  (segment (start 161.798 75.565) (end 161.798 77.47) (width 0.25) (layer F.Cu) (net 17))
+  (segment (start 161.798 77.47) (end 154.178 85.09) (width 0.25) (layer F.Cu) (net 17))
+  (segment (start 164.338 75.565) (end 164.338 77.47) (width 0.25) (layer F.Cu) (net 18))
+  (segment (start 164.338 77.47) (end 156.718 85.09) (width 0.25) (layer F.Cu) (net 18))
+  (segment (start 166.878 75.565) (end 166.878 81.661) (width 0.25) (layer F.Cu) (net 19))
+  (segment (start 153.797 87.249) (end 151.638 85.09) (width 0.25) (layer F.Cu) (net 19))
   (segment (start 161.29 87.249) (end 153.797 87.249) (width 0.25) (layer F.Cu) (net 19))
   (segment (start 166.878 81.661) (end 161.29 87.249) (width 0.25) (layer F.Cu) (net 19))
-  (segment (start 169.418 75.565) (end 169.418 81.661) (width 0.25) (layer F.Cu) (net 20) (status 400000))
-  (segment (start 152.781 88.773) (end 149.098 85.09) (width 0.25) (layer F.Cu) (net 20) (status 800000))
+  (segment (start 169.418 75.565) (end 169.418 81.661) (width 0.25) (layer F.Cu) (net 20))
+  (segment (start 152.781 88.773) (end 149.098 85.09) (width 0.25) (layer F.Cu) (net 20))
   (segment (start 162.306 88.773) (end 152.781 88.773) (width 0.25) (layer F.Cu) (net 20))
   (segment (start 169.418 81.661) (end 162.306 88.773) (width 0.25) (layer F.Cu) (net 20))
-  (segment (start 127.508 102.235) (end 127.508 106.68) (width 0.25) (layer F.Cu) (net 33) (status 400000))
-  (segment (start 127.508 106.68) (end 128.778 107.95) (width 0.25) (layer F.Cu) (net 33) (status 800000))
+  (segment (start 127.508 102.235) (end 127.508 106.68) (width 0.25) (layer F.Cu) (net 33))
+  (segment (start 127.508 106.68) (end 128.778 107.95) (width 0.25) (layer F.Cu) (net 33))
   (segment (start 144.018 85.09) (end 139.573 89.535) (width 0.25) (layer F.Cu) (net 34))
   (segment (start 139.573 92.71) (end 130.048 102.235) (width 0.25) (layer F.Cu) (net 34))
   (segment (start 139.573 89.535) (end 139.573 92.71) (width 0.25) (layer F.Cu) (net 34))
-  (segment (start 133.223 102.235) (end 133.223 106.68) (width 0.25) (layer F.Cu) (net 35) (status 400000))
-  (segment (start 133.223 106.68) (end 134.493 107.95) (width 0.25) (layer F.Cu) (net 35) (status 800000))
+  (segment (start 133.223 102.235) (end 133.223 106.68) (width 0.25) (layer F.Cu) (net 35))
+  (segment (start 133.223 106.68) (end 134.493 107.95) (width 0.25) (layer F.Cu) (net 35))
   (segment (start 141.478 92.71) (end 141.478 96.52) (width 0.25) (layer F.Cu) (net 36))
   (segment (start 141.478 96.52) (end 135.763 102.235) (width 0.25) (layer F.Cu) (net 36))
-  (segment (start 138.938 102.235) (end 138.938 106.68) (width 0.25) (layer F.Cu) (net 37) (status 400000))
-  (segment (start 138.938 106.68) (end 140.208 107.95) (width 0.25) (layer F.Cu) (net 37) (status 800000))
+  (segment (start 138.938 102.235) (end 138.938 106.68) (width 0.25) (layer F.Cu) (net 37))
+  (segment (start 138.938 106.68) (end 140.208 107.95) (width 0.25) (layer F.Cu) (net 37))
   (segment (start 144.018 92.71) (end 144.018 99.695) (width 0.25) (layer F.Cu) (net 38))
   (segment (start 144.018 99.695) (end 141.478 102.235) (width 0.25) (layer F.Cu) (net 38))
-  (segment (start 144.653 102.235) (end 144.653 106.68) (width 0.25) (layer F.Cu) (net 39) (status 400000))
-  (segment (start 144.653 106.68) (end 145.923 107.95) (width 0.25) (layer F.Cu) (net 39) (status 800000))
+  (segment (start 144.653 102.235) (end 144.653 106.68) (width 0.25) (layer F.Cu) (net 39))
+  (segment (start 144.653 106.68) (end 145.923 107.95) (width 0.25) (layer F.Cu) (net 39))
   (segment (start 146.558 92.71) (end 146.558 101.6) (width 0.25) (layer F.Cu) (net 40))
   (segment (start 146.558 101.6) (end 147.193 102.235) (width 0.25) (layer F.Cu) (net 40))
-  (segment (start 150.368 102.235) (end 150.368 106.68) (width 0.25) (layer F.Cu) (net 41) (status 400000))
-  (segment (start 150.368 106.68) (end 151.638 107.95) (width 0.25) (layer F.Cu) (net 41) (status 800000))
+  (segment (start 150.368 102.235) (end 150.368 106.68) (width 0.25) (layer F.Cu) (net 41))
+  (segment (start 150.368 106.68) (end 151.638 107.95) (width 0.25) (layer F.Cu) (net 41))
   (segment (start 149.098 92.71) (end 149.098 98.425) (width 0.25) (layer F.Cu) (net 42))
   (segment (start 149.098 98.425) (end 152.908 102.235) (width 0.25) (layer F.Cu) (net 42))
-  (segment (start 156.083 102.235) (end 156.083 106.68) (width 0.25) (layer F.Cu) (net 43) (status 400000))
-  (segment (start 156.083 106.68) (end 157.353 107.95) (width 0.25) (layer F.Cu) (net 43) (status 800000))
+  (segment (start 156.083 102.235) (end 156.083 106.68) (width 0.25) (layer F.Cu) (net 43))
+  (segment (start 156.083 106.68) (end 157.353 107.95) (width 0.25) (layer F.Cu) (net 43))
   (segment (start 151.638 92.71) (end 151.638 95.25) (width 0.25) (layer F.Cu) (net 44))
   (segment (start 151.638 95.25) (end 158.623 102.235) (width 0.25) (layer F.Cu) (net 44))
-  (segment (start 161.798 102.235) (end 161.798 106.68) (width 0.25) (layer F.Cu) (net 45) (status 400000))
-  (segment (start 161.798 106.68) (end 163.068 107.95) (width 0.25) (layer F.Cu) (net 45) (status 800000))
+  (segment (start 161.798 102.235) (end 161.798 106.68) (width 0.25) (layer F.Cu) (net 45))
+  (segment (start 161.798 106.68) (end 163.068 107.95) (width 0.25) (layer F.Cu) (net 45))
   (segment (start 154.178 92.71) (end 154.813 92.71) (width 0.25) (layer F.Cu) (net 46))
   (segment (start 154.813 92.71) (end 164.338 102.235) (width 0.25) (layer F.Cu) (net 46))
-  (segment (start 167.513 102.235) (end 167.513 106.68) (width 0.25) (layer F.Cu) (net 47) (status 400000))
-  (segment (start 167.513 106.68) (end 168.783 107.95) (width 0.25) (layer F.Cu) (net 47) (status 800000))
+  (segment (start 167.513 102.235) (end 167.513 106.68) (width 0.25) (layer F.Cu) (net 47))
+  (segment (start 167.513 106.68) (end 168.783 107.95) (width 0.25) (layer F.Cu) (net 47))
   (segment (start 156.718 92.71) (end 157.353 92.71) (width 0.25) (layer F.Cu) (net 48))
   (segment (start 157.353 92.71) (end 162.433 97.79) (width 0.25) (layer F.Cu) (net 48))

Commit message: updated readme
Parts:
- moved D3 1.63 mm to (140.2, 103.3), turned to 90 degrees
- moved D4 1.63 mm to (145.9, 103.3), turned to 90 degrees
- moved D5 1.63 mm to (151.6, 103.3), turned to 90 degrees
- moved D6 1.63 mm to (157.4, 103.3), turned to 90 degrees
- moved D7 1.63 mm to (163.1, 103.3), turned to 90 degrees
- moved D1 1.63 mm to (128.8, 103.3), turned to 90 degrees
- moved D2 1.63 mm to (134.5, 103.3), turned to 90 degrees
- moved D8 1.63 mm to (168.8, 103.3), turned to 90 degrees
Routing:
- net Net-(D6-Pad2): track 12.4 -> 10.4 mm
- net Net-(D5-Pad2): track 11.1 -> 9.05 mm
- net Net-(D7-Pad1): track 6.24 -> 4.70 mm
- net Net-(D6-Pad1): track 6.24 -> 4.70 mm
- net Net-(D5-Pad1): track 6.24 -> 4.70 mm
- net Net-(D4-Pad1): track 6.24 -> 4.70 mm
- net Net-(D3-Pad1): track 6.24 -> 4.70 mm
- net Net-(D1-Pad1): track 6.24 -> 4.70 mm
- net Net-(D8-Pad1): track 6.24 -> 4.70 mm
- net Net-(D2-Pad1): track 6.24 -> 4.70 mm
- net Net-(D4-Pad2): track 9.79 -> 8.26 mm
- net Net-(D8-Pad2): track 17.3 -> 16.0 mm
- net Net-(D7-Pad2): track 14.1 -> 13.0 mm
- net Net-(D2-Pad2): track 11.9 -> 10.9 mm
- net Net-(D3-Pad2): track 10.6 -> 9.58 mm
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